Commit message: Final changes stashed

File: urdf/sim.xacro (robot description, xacro)
@@ -1,50 +1,65 @@
 <?xml version="1.0"?>
-<robot xmlns:xacro="http://www.ros.org/wiki/xacro" name="sim_loader">
+<robot name="sim_loader" xmlns:xacro="http://www.ros.org/wiki/xacro">
   <gazebo>
-    <plugin name="ros_control" filename="libgazebo_ros_control.so">
+    <plugin filename="libgazebo_ros_control.so" name="ros_control">
       <robotNamespace>/asv</robotNamespace>
       <robotSimType>gazebo_ros_control/DefaultRobotHWSim</robotSimType>
     </plugin>
   </gazebo>
-  <gazebo reference="asv_description">
-    <plugin name="water_dynamics" filename="libusv_gazebo_dynamics_plugin.so">
-    <bodyName>base_footprint</bodyName>
-    <waterLevel>.05</waterLevel>
-    <waterDensity>997.8</waterDensity>
-    <cmdTimeout>1.0</cmdTimeout>
-    <xDotU>5.0</xDotU>
-    <yDotV>5.0</yDotV>
-    <nDotR>1.0</nDotR>
-    <xU>20.0</xU>
-    <xUU>0.0</xUU>
-    <yV>20.0</yV>
-    <yVV>0.0</yVV>
-    <zW>50.0</zW>
-    <kP>10.0</kP>
-    <mQ>10.0</mQ>
-    <nR>20.0</nR>
-    <nRR>0.0</nRR>
-    <maxCmd>1.0</maxCmd>
-    <maxForceFwd>100.0</maxForceFwd>
-    <maxForceRev>-80.0</maxForceRev>
-    <boatArea>0.48</boatArea>
-    <boatWidth>1.0</boatWidth>
-    <boatLength>1.35</boatLength>
-    <thrustOffsetZ>-0.01</thrustOffsetZ>
-    <metacentricLength>0.4</metacentricLength>
-    <metacentricWidth>0.4</metacentricWidth>
-  </plugin>
-</gazebo>
+  <!--<gazebo reference="asv_description">
+    <plugin filename="libusv_gazebo_dynamics_plugin.so" name="water_dynamics">
+      <bodyName>base_footprint</bodyName>
+      <waterLevel>.05</waterLevel>
+      <waterDensity>997.8</waterDensity>
+      <cmdTimeout>1.0</cmdTimeout>
+      <xDotU>5.0</xDotU>
+      <yDotV>5.0</yDotV>
+      <nDotR>1.0</nDotR>
+      <xU>20.0</xU>
+      <xUU>0.0</xUU>
+      <yV>20.0</yV>
+      <yVV>0.0</yVV>
+      <zW>50.0</zW>
+      <kP>10.0</kP>
+      <mQ>10.0</mQ>
+      <nR>20.0</nR>
+      <nRR>0.0</nRR>
+      <maxCmd>1.0</maxCmd>
+      <maxForceFwd>100.0</maxForceFwd>
+      <maxForceRev>-80.0</maxForceRev>
+      <boatArea>0.48</boatArea>
+      <boatWidth>1.0</boatWidth>
+      <boatLength>1.35</boatLength>
+      <thrustOffsetZ>-0.01</thrustOffsetZ>
+      <metacentricLength>0.4</metacentricLength>
+      <metacentricWidth>0.4</metacentricWidth>
+    </plugin>
+  </gazebo>-->
   <gazebo>
-    <plugin name="controller" filename="libthruster_controller.so" />
+    <plugin filename="libgazebo_ros_force.so" name="gazebo_ros_force">
+      <alwaysOn>1</alwaysOn>
+      <bodyName>thruster_left</bodyName>
+      <topicName>left_force</topicName>
+      <robotNamespace>asv</robotNamespace>
+    </plugin>
+    <plugin filename="libgazebo_ros_force.so" name="gazebo_ros_force">
+      <alwaysOn>1</alwaysOn>
+      <bodyName>thruster_right</bodyName>
+      <topicName>right_force</topicName>
+      <robotNamespace>asv</robotNamespace>
+    </plugin>
+  </gazebo>
+  <gazebo>
+    <plugin name="BuoyancyPlugin" filename="libBuoyancyPlugin.so">
+      <fluid_density>997.8</fluid_density>
+      <link name="base_link" />
+    </plugin>
   </gazebo>
   <!--<gazebo>
-    <plugin name="asv_controller" filename="libgazebo_ros_planar_move.so">
-      <commandTopic>cmd_vel</commandTopic>
-      <odometryTopic>odom</odometryTopic>
-      <odometryFrame>odom</odometryFrame>
-      <odometryRate>100.0</odometryRate>
-      <robotBaseFrame>base_footprint</robotBaseFrame>
+    <plugin filename="libthruster_control.so" name="controller">
+      <bodyName>base_link</bodyName>
+      <topicName>force</topicName>
     </plugin>
   </gazebo>-->
+  <!--<gazebo><plugin name="asv_controller" filename="libgazebo_ros_planar_move.so"><commandTopic>cmd_vel</commandTopic><odometryTopic>odom</odometryTopic><odometryFrame>odom</odometryFrame><odometryRate>100.0</odometryRate><robotBaseFrame>base_footprint</robotBaseFrame></plugin></gazebo>-->
 </robot>
