Commit message: Stashing commits before modifying local system

File: urdf/asv_sensors.xacro (robot description, xacro)
@@ -2,16 +2,17 @@
 <robot name="sensors" xmlns:xacro="http://www.ros.org/wiki/xacro">
 	<sensor name="lidar" type="laser" update_rate="50">
-		<parent link="lidar"/>
+		<parent link="base_link"/>
 		<origin rpy="0 0 0" xyz="0 0 0"/>
+		<update_rate>50</update_rate>
 	</sensor>
-	<!--<gazebo reference="lidar">
+	<gazebo reference="base_link">
 		<sensor name="lmssick" type="ray">s
 			<ray>
 				<scan>
 					<horizontal>
-						<samples>100</samples>
-						<resolution>1</resolution>
-						<min_angle>-1.1781</min_angle>
-						<max_angle>1.1781</max_angle></horizontal>
+						<samples>540</samples>
+						<resolution>0.5</resolution>
+						<min_angle>-${3*PI/4}</min_angle>
+						<max_angle>${3*PI/4}</max_angle></horizontal>
 					<vertical>
 						<samples>1</samples>
@@ -23,5 +24,5 @@
 				<range>
 					<min>0.5</min>
-					<max>20</max>
+					<max>50</max>
 					<resolution>1</resolution>
 				</range>
@@ -33,15 +34,15 @@
 			</ray>
 			<plugin filename="libgazebo_ros_laser.so" name="lidar">
-				<topicName>/asv/laser/scan</topicName>
-				<frameName>lidar</frameName>
+				<topicName>/scan</topicName>
+				<frameName>base_link</frameName>
       			<visualize>true</visualize>
 			</plugin>
 		</sensor>
-	</gazebo>-->
-	<sensor name="camera" type="camera" update_rate="30">
-		<parent link="camera"/>
+	</gazebo>
+	<!--<sensor name="camera" type="camera" update_rate="30">
+		<parent link="base_link"/>
 		<origin rpy="0 0 0" xyz="0 0 0"/>
 	</sensor>
-	<gazebo reference="camera">
+	<gazebo reference="base_link">
 		<sensor name="camera1" type="camera">
 			<camera name="cam_head">
@@ -76,9 +77,8 @@
 			</plugin>
 		</sensor>
-	</gazebo>
+	</gazebo>-->
 	<gazebo>
 			<plugin filename="libhector_gazebo_ros_imu.so" name="imu_plugin">
-				<updateRate>100</updateRate>
-				<robotNamespace>asv</robotNamespace>
+				<updateRate>20</updateRate>
 				<bodyName>base_link</bodyName>
 				<topicName>imu_data</topicName>
@@ -93,6 +93,6 @@
 				<yawDrift>0</yawDrift>
 				<yawDriftFrequency>0</yawDriftFrequency>
-				<yawGaussianNoise>0</yawGaussianNoise>
-				<gaussianNoise>0.0</gaussianNoise>
+				<yawGaussianNoise>0.000</yawGaussianNoise>
+				<gaussianNoise>0.000</gaussianNoise>
 				<rpyOffset>0 0 0</rpyOffset>
 				<xyzOffset>0 0 0</xyzOffset>
@@ -102,12 +102,12 @@
 		<!--Be careful of Plugins that are for models and that are for links and for worlds.-->
 			<plugin filename="libhector_gazebo_ros_gps.so" name="gps_sim">
-				<updateRate>100</updateRate>
-				<bodyName>garmin</bodyName>
+				<updateRate>10</updateRate>
+				<bodyName>base_link</bodyName>
 				<topicName>/fix</topicName>
 				<velocityTopicName>/vel</velocityTopicName>
-				<drift>5.0 5.0 5.0</drift>
-				<gaussianNoise>0.1 0.1 0.1</gaussianNoise>
+				<drift>0 0 0</drift>
+				<gaussianNoise>0.000 0.000 0.000</gaussianNoise>
 				<velocityDrift>0 0 0</velocityDrift>
-				<velocityGaussianNoise>0.1 0.1 0.1</velocityGaussianNoise>
+				<velocityGaussianNoise>0 0 0</velocityGaussianNoise>
 			</plugin>
 	</gazebo>

File: urdf/gazebo.xacro (robot description, xacro)
@@ -1,4 +1,5 @@
 <?xml version="1.0"?>
 <robot name="asv_gazebo" xmlns:xacro="http://www.ros.org/wiki/xacro">
+  	<xacro:include filename="$(find asv_description)/urdf/common_properties.xacro"/>
 	<xacro:include filename="$(find asv_gazebo)/urdf/sim.xacro"/>
 	<xacro:include filename="$(find asv_gazebo)/urdf/asv_sensors.xacro"/>

File: urdf/sim.xacro (robot description, xacro)
@@ -7,8 +7,8 @@
     </plugin>
   </gazebo>
-  <!--<gazebo reference="asv_description">
+  <gazebo reference="asv_description">
     <plugin filename="libusv_gazebo_dynamics_plugin.so" name="water_dynamics">
-      <bodyName>base_footprint</bodyName>
-      <waterLevel>.05</waterLevel>
+      <bodyName>base_link</bodyName>
+      <waterLevel>0.05</waterLevel>
       <waterDensity>997.8</waterDensity>
       <cmdTimeout>1.0</cmdTimeout>
@@ -35,33 +35,17 @@
       <metacentricWidth>0.4</metacentricWidth>
     </plugin>
-  </gazebo>-->
+  </gazebo>
   <gazebo>
-    <plugin filename="libthruster_control.so" name="gazebo_ros_force">
-      <alwaysOn>1</alwaysOn>
-      <bodyName>base_footprint</bodyName>
-      <LeftThrusterName>thruster_left</LeftThrusterName>
-      <RightThrusterName>thruster_right</RightThrusterName>
+    <plugin name="gazebo_thruster_control" filename="libthruster_control.so">
+      <bodyName>base_hull</bodyName>
       <LeftTopicName>/left_pwm</LeftTopicName>
       <RightTopicName>/right_pwm</RightTopicName>
     </plugin>
   </gazebo>
-    <!--<plugin filename="libthruster_control.so" name="gazebo_ros_force">
-      <alwaysOn>1</alwaysOn>
-      <bodyName>base_link</bodyName>
-      <topicName>/right_pwm</topicName>
-    </plugin>
+  <!--<gazebo reference="base_hull">
+    <gravity>0</gravity>
+  </gazebo>
+  <gazebo reference="base_link">
+    <gravity>0</gravity>
   </gazebo>-->
-  <!--<gazebo>
-    <plugin name="BuoyancyPlugin" filename="libBuoyancyPlugin.so">
-      <fluid_density>997.8</fluid_density>
-      <link name="base_link" />
-    </plugin>
-  </gazebo>-->
-  <!--<gazebo>
-    <plugin filename="libthruster_control.so" name="controller">
-      <bodyName>base_link</bodyName>
-      <topicName>force</topicName>
-    </plugin>
-  </gazebo>-->
-  <!--<gazebo><plugin name="asv_controller" filename="libgazebo_ros_planar_move.so"><commandTopic>cmd_vel</commandTopic><odometryTopic>odom</odometryTopic><odometryFrame>odom</odometryFrame><odometryRate>100.0</odometryRate><robotBaseFrame>base_footprint</robotBaseFrame></plugin></gazebo>-->
 </robot>

Commit message: Fixed common issues

File: urdf/asv_sensors.xacro (robot description, xacro)
@@ -2,9 +2,9 @@
 <robot name="sensors" xmlns:xacro="http://www.ros.org/wiki/xacro">
 	<sensor name="lidar" type="laser" update_rate="50">
-		<parent link="base_link"/>
+		<parent link="lidar"/>
 		<origin rpy="0 0 0" xyz="0 0 0"/>
 		<update_rate>50</update_rate>
 	</sensor>
-	<gazebo reference="base_link">
+	<gazebo reference="lidar">
 		<sensor name="lmssick" type="ray">s
 			<ray>
@@ -35,14 +35,14 @@
 			<plugin filename="libgazebo_ros_laser.so" name="lidar">
 				<topicName>/scan</topicName>
-				<frameName>base_link</frameName>
+				<frameName>lidar</frameName>
       			<visualize>true</visualize>
 			</plugin>
 		</sensor>
 	</gazebo>
-	<!--<sensor name="camera" type="camera" update_rate="30">
-		<parent link="base_link"/>
+	<sensor name="camera" type="camera" update_rate="30">
+		<parent link="lidar"/>
 		<origin rpy="0 0 0" xyz="0 0 0"/>
 	</sensor>
-	<gazebo reference="base_link">
+	<gazebo reference="lidar">
 		<sensor name="camera1" type="camera">
 			<camera name="cam_head">
@@ -64,9 +64,9 @@
 			</camera>
 			<plugin filename="libgazebo_ros_camera.so" name="camera_controller">
-				<robotNamespace>asv</robotNamespace>
+				<robotNamespace>/</robotNamespace>
 				<cameraName>camera</cameraName>
 				<imageTopicName>image_raw</imageTopicName>
 				<cameraInfoTopicName>camera_info</cameraInfoTopicName>
-				<frameName>camera</frameName>
+				<frameName>lidar</frameName>
 				<hackBaseline>0.07</hackBaseline>
 				<distortionK1>0.0</distortionK1>
@@ -77,22 +77,11 @@
 			</plugin>
 		</sensor>
-	</gazebo>-->
+	</gazebo>
 	<gazebo>
-			<plugin filename="libhector_gazebo_ros_imu.so" name="imu_plugin">
+			<plugin filename="libgazebo_ros_imu.so" name="imu_plugin">
 				<updateRate>20</updateRate>
 				<bodyName>base_link</bodyName>
 				<topicName>imu_data</topicName>
-				<accelOffset>0 0 0</accelOffset>
-				<accelDrift>0 0 0</accelDrift>
-				<accelDriftFrequency>0 0 0</accelDriftFrequency>
-				<rateOffset>0 0 0</rateOffset>
-				<rateDrift>0 0 0</rateDrift>
-				<rateDriftFrequency>0 0 0</rateDriftFrequency>
-				<rateGuassianNoise>0 0 0</rateGuassianNoise>
-				<yawOffset>0</yawOffset>
-				<yawDrift>0</yawDrift>
-				<yawDriftFrequency>0</yawDriftFrequency>
-				<yawGaussianNoise>0.000</yawGaussianNoise>
-				<gaussianNoise>0.000</gaussianNoise>
+				<gaussianNoise>0.0001</gaussianNoise>
 				<rpyOffset>0 0 0</rpyOffset>
 				<xyzOffset>0 0 0</xyzOffset>
@@ -104,6 +93,18 @@
 				<updateRate>10</updateRate>
 				<bodyName>base_link</bodyName>
-				<topicName>/fix</topicName>
-				<velocityTopicName>/vel</velocityTopicName>
+				<topicName>/boat_fix</topicName>
+				<velocityTopicName>/boat_vel</velocityTopicName>
+				<drift>0 0 0</drift>
+				<gaussianNoise>0.000 0.000 0.000</gaussianNoise>
+				<velocityDrift>0 0 0</velocityDrift>
+				<velocityGaussianNoise>0 0 0</velocityGaussianNoise>
+			</plugin>
+	</gazebo>
+	<gazebo>
+			<plugin filename="libhector_gazebo_ros_gps.so" name="gps_base">
+				<updateRate>10</updateRate>
+				<bodyName>base_link</bodyName>
+				<topicName>/base_fix</topicName>
+				<velocityTopicName>/base_vel</velocityTopicName>
 				<drift>0 0 0</drift>
 				<gaussianNoise>0.000 0.000 0.000</gaussianNoise>
